File: kicad/traffic_lights/lcd_module.sch (KiCad schematic (older format))
At the start: 5 parts

Commit message: update..
Parts:
- gave numbers to parts that had none: 5
Changed lines of the file:
@@
 $Descr A4 11693 8268
 encoding utf-8
-Sheet 3 4
+Sheet 3 5
 Title ""
 Date "24 jun 2015"
@@
 $EndDescr
 $Comp
-L RC1602A-GHW-ESX DS?
+L RC1602A-GHW-ESX DS1
 U 1 1 558A7AA4
 P 4700 1950
-F 0 "DS?" H 3900 2350 40  0000 C CNN
+F 0 "DS1" H 3900 2350 40  0000 C CNN
 F 1 "RC1602A-GHW-ESX" H 5250 2350 40  0000 C CNN
 F 2 "RC1602A" H 4700 1900 35  0000 C CIN
@@
 $EndComp
 $Comp
-L GND #PWR?
+L GND #PWR046
 U 1 1 558A7AB3
 P 5450 2550
-F 0 "#PWR?" H 5450 2550 30  0001 C CNN
+F 0 "#PWR046" H 5450 2550 30  0001 C CNN
 F 1 "GND" H 5450 2480 30  0001 C CNN
 F 2 "" H 5450 2550 60  0000 C CNN
@@
 $EndComp
 $Comp
-L GND #PWR?
+L GND #PWR047
 U 1 1 558A7AC2
 P 3950 2550
-F 0 "#PWR?" H 3950 2550 30  0001 C CNN
+F 0 "#PWR047" H 3950 2550 30  0001 C CNN
 F 1 "GND" H 3950 2480 30  0001 C CNN
 F 2 "" H 3950 2550 60  0000 C CNN
@@
 $EndComp
 $Comp
-L VCC #PWR?
+L VCC #PWR048
 U 1 1 558A7ADE
 P 5350 3150
-F 0 "#PWR?" H 5350 3250 30  0001 C CNN
+F 0 "#PWR048" H 5350 3250 30  0001 C CNN
 F 1 "VCC" H 5350 3250 30  0000 C CNN
 F 2 "" H 5350 3150 60  0000 C CNN
@@
 $EndComp
 $Comp
-L VCC #PWR?
+L VCC #PWR049
 U 1 1 558A7AED
 P 4050 2550
-F 0 "#PWR?" H 4050 2650 30  0001 C CNN
+F 0 "#PWR049" H 4050 2650 30  0001 C CNN
 F 1 "VCC" H 4050 2650 30  0000 C CNN
 F 2 "" H 4050 2550 60  0000 C CNN
@@
 $EndComp
 $Comp
-L R R?
+L R R11
 U 1 1 558A7B10
 P 5400 2900
-F 0 "R?" V 5480 2900 40  0000 C CNN
+F 0 "R11" V 5480 2900 40  0000 C CNN
 F 1 "1k" V 5407 2901 40  0000 C CNN
 F 2 "~" V 5330 2900 30  0000 C CNN
@@
 $EndComp
 $Comp
-L POT RV?
+L POT RV5
 U 1 1 558A7B68
 P 4150 3000
-F 0 "RV?" H 4150 2900 50  0000 C CNN
+F 0 "RV5" H 4150 2900 50  0000 C CNN
 F 1 "10k" H 4150 3000 50  0000 C CNN
 F 2 "~" H 4150 3000 60  0000 C CNN
@@
 $EndComp
 $Comp
-L VCC #PWR?
+L VCC #PWR050
 U 1 1 558A7B77
 P 3800 2900
-F 0 "#PWR?" H 3800 3000 30  0001 C CNN
+F 0 "#PWR050" H 3800 3000 30  0001 C CNN
 F 1 "VCC" H 3800 3000 30  0000 C CNN
 F 2 "" H 3800 2900 60  0000 C CNN
@@
 $EndComp
 $Comp
-L GND #PWR?
+L GND #PWR051
 U 1 1 558A7B86
 P 4500 3100
-F 0 "#PWR?" H 4500 3100 30  0001 C CNN
+F 0 "#PWR051" H 4500 3100 30  0001 C CNN
 F 1 "GND" H 4500 3030 30  0001 C CNN
 F 2 "" H 4500 3100 60  0000 C CNN
@@
 $EndComp
 $Comp
-L GND #PWR?
+L GND #PWR052
 U 1 1 558A7BB7
 P 4350 2550
-F 0 "#PWR?" H 4350 2550 30  0001 C CNN
+F 0 "#PWR052" H 4350 2550 30  0001 C CNN
 F 1 "GND" H 4350 2480 30  0001 C CNN
 F 2 "" H 4350 2550 60  0000 C CNN
@@
 LCD_LATCH_ENABLE
 $Comp
-L 74HC595N IC?
+L 74HC595N IC2
 U 1 1 558AE170
 P 6900 2650
-F 0 "IC?" H 6600 3175 50  0000 L BNN
+F 0 "IC2" H 6600 3175 50  0000 L BNN
 F 1 "74HC595N" H 6600 1950 50  0000 L BNN
 F 2 "74xx-eu-DIL16" V 6900 2600 50  0001 C CNN
@@
 $EndComp
 $Comp
-L GND #PWR?
+L GND #PWR053
 U 1 1 558AE193
 P 7500 2250
-F 0 "#PWR?" H 7500 2250 30  0001 C CNN
+F 0 "#PWR053" H 7500 2250 30  0001 C CNN
 F 1 "GND" H 7500 2180 30  0001 C CNN
 F 2 "" H 7500 2250 60  0000 C CNN
@@
 LCD_SR_RESET
 $Comp
-L CONNECTOR_6_PIN CON?
+L CONNECTOR_6_PIN CON1
 U 1 1 558AE8CB
 P 9100 1950
-F 0 "CON?" V 9750 1400 50  0000 L BNN
+F 0 "CON1" V 9750 1400 50  0000 L BNN
 F 1 "CONNECTOR_6_PIN" H 8800 1250 50  0000 L BNN
 F 2 "CON6x1" V 9100 1900 50  0001 C CNN
@@
 	5750 3400 5750 1900
 Wire Wire Line
-	5750 1900 7550 1900
-Wire Wire Line
-	7550 1900 7650 1900
+	5750 1900 7650 1900
 Wire Wire Line
 	7400 2150 7500 2150
@@
 	7500 2150 7500 2250
 Wire Wire Line
-	7650 2550 7550 2550
-Wire Wire Line
-	7550 2550 7400 2550
-Wire Wire Line
-	7400 2850 7550 2850
-Wire Wire Line
-	7550 2850 7650 2850
-Wire Wire Line
-	7400 3050 7550 3050
-Wire Wire Line
-	7550 3050 7650 3050
-Wire Wire Line
-	7400 2700 7550 2700
-Wire Wire Line
-	7550 2700 7650 2700
+	7400 2550 7650 2550
+Wire Wire Line
+	7400 2850 7650 2850
+Wire Wire Line
+	7400 3050 7650 3050
+Wire Wire Line
+	7400 2700 7650 2700
 Wire Wire Line
 	8800 1700 8800 2650
