File: kicad/traffic_lights/traffic_light_leds.sch (KiCad schematic (older format))
At the start: 34 parts

Commit message: update..
Parts:
- gave numbers to parts that had none: 34
Changed lines of the file:
@@
 $Descr A4 11693 8268
 encoding utf-8
-Sheet 4 4
+Sheet 4 5
 Title ""
 Date "24 jun 2015"
@@
 $EndDescr
 $Comp
-L 74AC164N IC?
+L 74AC164N IC3
 U 1 1 558B35E2
 P 7450 2750
-F 0 "IC?" H 7150 3175 50  0000 L BNN
+F 0 "IC3" H 7150 3175 50  0000 L BNN
 F 1 "74AC164N" H 7150 2150 50  0000 L BNN
 F 2 "74xx-eu-DIL14" H 7450 2900 50  0001 C CNN
@@
 $EndComp
 $Comp
-L 74AC164N IC?
+L 74AC164N IC4
 U 1 1 558B35EF
 P 7450 4050
-F 0 "IC?" H 7150 4475 50  0000 L BNN
+F 0 "IC4" H 7150 4475 50  0000 L BNN
 F 1 "74AC164N" H 7150 3450 50  0000 L BNN
 F 2 "74xx-eu-DIL14" H 7450 4200 50  0001 C CNN
@@
 $EndComp
 $Comp
-L LED D?
+L LED D10
 U 1 1 558B35F7
 P 4450 1450
-F 0 "D?" H 4450 1550 50  0000 C CNN
+F 0 "D10" H 4450 1550 50  0000 C CNN
 F 1 "LED" H 4450 1350 50  0000 C CNN
 F 2 "~" H 4450 1450 60  0000 C CNN
@@
 $EndComp
 $Comp
-L LED D?
+L LED D11
 U 1 1 558B3622
 P 4450 1600
-F 0 "D?" H 4450 1700 50  0000 C CNN
+F 0 "D11" H 4450 1700 50  0000 C CNN
 F 1 "LED" H 4450 1500 50  0000 C CNN
 F 2 "~" H 4450 1600 60  0000 C CNN
@@
 $EndComp
 $Comp
-L LED D?
+L LED D12
 U 1 1 558B3628
 P 4450 1750
-F 0 "D?" H 4450 1850 50  0000 C CNN
+F 0 "D12" H 4450 1850 50  0000 C CNN
 F 1 "LED" H 4450 1650 50  0000 C CNN
 F 2 "~" H 4450 1750 60  0000 C CNN
@@
 $EndComp
 $Comp
-L LED D?
+L LED D13
 U 1 1 558B362E
 P 4450 1900
-F 0 "D?" H 4450 2000 50  0000 C CNN
+F 0 "D13" H 4450 2000 50  0000 C CNN
 F 1 "LED" H 4450 1800 50  0000 C CNN
 F 2 "~" H 4450 1900 60  0000 C CNN
@@
 $EndComp
 $Comp
-L R R?
+L R R12
 U 1 1 558B3636
 P 5000 1450
-F 0 "R?" V 5080 1450 40  0000 C CNN
+F 0 "R12" V 5080 1450 40  0000 C CNN
 F 1 "1k" V 5007 1451 40  0000 C CNN
 F 2 "~" V 4930 1450 30  0000 C CNN
@@
 $EndComp
 $Comp
-L R R?
+L R R13
 U 1 1 558B365C
 P 5000 1600
-F 0 "R?" V 5080 1600 40  0000 C CNN
+F 0 "R13" V 5080 1600 40  0000 C CNN
 F 1 "1k" V 5007 1601 40  0000 C CNN
 F 2 "~" V 4930 1600 30  0000 C CNN
@@
 $EndComp
 $Comp
-L R R?
+L R R14
 U 1 1 558B3662
 P 5000 1750
-F 0 "R?" V 5080 1750 40  0000 C CNN
+F 0 "R14" V 5080 1750 40  0000 C CNN
 F 1 "1k" V 5007 1751 40  0000 C CNN
 F 2 "~" V 4930 1750 30  0000 C CNN
@@
 $EndComp
 $Comp
-L VCC #PWR?
+L VCC #PWR054
 U 1 1 558B3688
 P 4100 1300
-F 0 "#PWR?" H 4100 1400 30  0001 C CNN
+F 0 "#PWR054" H 4100 1400 30  0001 C CNN
 F 1 "VCC" H 4100 1400 30  0000 C CNN
 F 2 "" H 4100 1300 60  0000 C CNN
@@
 $EndComp
 $Comp
-L R R?
+L R R15
 U 1 1 558B3668
 P 5000 1900
-F 0 "R?" V 5080 1900 40  0000 C CNN
+F 0 "R15" V 5080 1900 40  0000 C CNN
 F 1 "1k" V 5007 1901 40  0000 C CNN
 F 2 "~" V 4930 1900 30  0000 C CNN
@@
 $EndComp
 $Comp
-L LED D?
+L LED D14
 U 1 1 558B3895
 P 4450 2550
-F 0 "D?" H 4450 2650 50  0000 C CNN
+F 0 "D14" H 4450 2650 50  0000 C CNN
 F 1 "LED" H 4450 2450 50  0000 C CNN
 F 2 "~" H 4450 2550 60  0000 C CNN
@@
 $EndComp
 $Comp
-L LED D?
+L LED D15
 U 1 1 558B389B
 P 4450 2700
-F 0 "D?" H 4450 2800 50  0000 C CNN
+F 0 "D15" H 4450 2800 50  0000 C CNN
 F 1 "LED" H 4450 2600 50  0000 C CNN
 F 2 "~" H 4450 2700 60  0000 C CNN
@@
 $EndComp
 $Comp
-L LED D?
+L LED D16
 U 1 1 558B38A1
 P 4450 2850
-F 0 "D?" H 4450 2950 50  0000 C CNN
+F 0 "D16" H 4450 2950 50  0000 C CNN
 F 1 "LED" H 4450 2750 50  0000 C CNN
 F 2 "~" H 4450 2850 60  0000 C CNN
@@
 $EndComp
 $Comp
-L LED D?
+L LED D17
 U 1 1 558B38A7
 P 4450 3000
-F 0 "D?" H 4450 3100 50  0000 C CNN
+F 0 "D17" H 4450 3100 50  0000 C CNN
 F 1 "LED" H 4450 2900 50  0000 C CNN
 F 2 "~" H 4450 3000 60  0000 C CNN
@@
 $EndComp
 $Comp
-L R R?
+L R R16
 U 1 1 558B38AD
 P 5000 2550
-F 0 "R?" V 5080 2550 40  0000 C CNN
+F 0 "R16" V 5080 2550 40  0000 C CNN
 F 1 "1k" V 5007 2551 40  0000 C CNN
 F 2 "~" V 4930 2550 30  0000 C CNN
@@
 $EndComp
 $Comp
-L R R?
+L R R17
 U 1 1 558B38B3
 P 5000 2700
-F 0 "R?" V 5080 2700 40  0000 C CNN
+F 0 "R17" V 5080 2700 40  0000 C CNN
 F 1 "1k" V 5007 2701 40  0000 C CNN
 F 2 "~" V 4930 2700 30  0000 C CNN
@@
 $EndComp
 $Comp
-L R R?
+L R R18
 U 1 1 558B38B9
 P 5000 2850
-F 0 "R?" V 5080 2850 40  0000 C CNN
+F 0 "R18" V 5080 2850 40  0000 C CNN
 F 1 "1k" V 5007 2851 40  0000 C CNN
 F 2 "~" V 4930 2850 30  0000 C CNN
@@
 $EndComp
 $Comp
-L VCC #PWR?
+L VCC #PWR055
 U 1 1 558B38BF
 P 4100 2400
-F 0 "#PWR?" H 4100 2500 30  0001 C CNN
+F 0 "#PWR055" H 4100 2500 30  0001 C CNN
 F 1 "VCC" H 4100 2500 30  0000 C CNN
 F 2 "" H 4100 2400 60  0000 C CNN
@@
 $EndComp
 $Comp
-L R R?
+L R R19
 U 1 1 558B38D6
 P 5000 3000
-F 0 "R?" V 5080 3000 40  0000 C CNN
+F 0 "R19" V 5080 3000 40  0000 C CNN
 F 1 "1k" V 5007 3001 40  0000 C CNN
 F 2 "~" V 4930 3000 30  0000 C CNN
@@
 $EndComp
 $Comp
-L LED D?
+L LED D18
 U 1 1 558B38DC
 P 4450 3700
-F 0 "D?" H 4450 3800 50  0000 C CNN
+F 0 "D18" H 4450 3800 50  0000 C CNN
 F 1 "LED" H 4450 3600 50  0000 C CNN
 F 2 "~" H 4450 3700 60  0000 C CNN
@@
 $EndComp
 $Comp
-L LED D?
+L LED D19
 U 1 1 558B38E2
 P 4450 3850
-F 0 "D?" H 4450 3950 50  0000 C CNN
+F 0 "D19" H 4450 3950 50  0000 C CNN
 F 1 "LED" H 4450 3750 50  0000 C CNN
 F 2 "~" H 4450 3850 60  0000 C CNN
@@
 $EndComp
 $Comp
-L LED D?
+L LED D20
 U 1 1 558B38E8
 P 4450 4000
-F 0 "D?" H 4450 4100 50  0000 C CNN
+F 0 "D20" H 4450 4100 50  0000 C CNN
 F 1 "LED" H 4450 3900 50  0000 C CNN
 F 2 "~" H 4450 4000 60  0000 C CNN
@@
 $EndComp
 $Comp
-L LED D?
+L LED D21
 U 1 1 558B38EE
 P 4450 4150
-F 0 "D?" H 4450 4250 50  0000 C CNN
+F 0 "D21" H 4450 4250 50  0000 C CNN
 F 1 "LED" H 4450 4050 50  0000 C CNN
 F 2 "~" H 4450 4150 60  0000 C CNN
@@
 $EndComp
 $Comp
-L R R?
+L R R20
 U 1 1 558B38F4
 P 5000 3700
-F 0 "R?" V 5080 3700 40  0000 C CNN
+F 0 "R20" V 5080 3700 40  0000 C CNN
 F 1 "1k" V 5007 3701 40  0000 C CNN
 F 2 "~" V 4930 3700 30  0000 C CNN
@@
 $EndComp
 $Comp
-L R R?
+L R R21
 U 1 1 558B38FA
 P 5000 3850
-F 0 "R?" V 5080 3850 40  0000 C CNN
+F 0 "R21" V 5080 3850 40  0000 C CNN
 F 1 "1k" V 5007 3851 40  0000 C CNN
 F 2 "~" V 4930 3850 30  0000 C CNN
@@
 $EndComp
 $Comp
-L R R?
+L R R22
 U 1 1 558B3900
 P 5000 4000
-F 0 "R?" V 5080 4000 40  0000 C CNN
+F 0 "R22" V 5080 4000 40  0000 C CNN
 F 1 "1k" V 5007 4001 40  0000 C CNN
 F 2 "~" V 4930 4000 30  0000 C CNN
@@
 $EndComp
 $Comp
-L VCC #PWR?
+L VCC #PWR056
 U 1 1 558B3906
 P 4100 3550
-F 0 "#PWR?" H 4100 3650 30  0001 C CNN
+F 0 "#PWR056" H 4100 3650 30  0001 C CNN
 F 1 "VCC" H 4100 3650 30  0000 C CNN
 F 2 "" H 4100 3550 60  0000 C CNN
@@
 $EndComp
 $Comp
-L R R?
+L R R23
 U 1 1 558B391D
 P 5000 4150
-F 0 "R?" V 5080 4150 40  0000 C CNN
+F 0 "R23" V 5080 4150 40  0000 C CNN
 F 1 "1k" V 5007 4151 40  0000 C CNN
 F 2 "~" V 4930 4150 30  0000 C CNN
@@
 $EndComp
 $Comp
-L LED D?
+L LED D22
 U 1 1 558B3923
 P 4450 4850
-F 0 "D?" H 4450 4950 50  0000 C CNN
+F 0 "D22" H 4450 4950 50  0000 C CNN
 F 1 "LED" H 4450 4750 50  0000 C CNN
 F 2 "~" H 4450 4850 60  0000 C CNN
@@
 $EndComp
 $Comp
-L LED D?
+L LED D23
 U 1 1 558B3929
 P 4450 5000
-F 0 "D?" H 4450 5100 50  0000 C CNN
+F 0 "D23" H 4450 5100 50  0000 C CNN
 F 1 "LED" H 4450 4900 50  0000 C CNN
 F 2 "~" H 4450 5000 60  0000 C CNN
@@
 $EndComp
 $Comp
-L LED D?
+L LED D24
 U 1 1 558B392F
 P 4450 5150
-F 0 "D?" H 4450 5250 50  0000 C CNN
+F 0 "D24" H 4450 5250 50  0000 C CNN
 F 1 "LED" H 4450 5050 50  0000 C CNN
 F 2 "~" H 4450 5150 60  0000 C CNN
@@
 $EndComp
 $Comp
-L LED D?
+L LED D25
 U 1 1 558B3935
 P 4450 5300
-F 0 "D?" H 4450 5400 50  0000 C CNN
+F 0 "D25" H 4450 5400 50  0000 C CNN
 F 1 "LED" H 4450 5200 50  0000 C CNN
 F 2 "~" H 4450 5300 60  0000 C CNN
@@
 $EndComp
 $Comp
-L R R?
+L R R24
 U 1 1 558B393B
 P 5000 4850
-F 0 "R?" V 5080 4850 40  0000 C CNN
+F 0 "R24" V 5080 4850 40  0000 C CNN
 F 1 "1k" V 5007 4851 40  0000 C CNN
 F 2 "~" V 4930 4850 30  0000 C CNN
@@
 $EndComp
 $Comp
-L R R?
+L R R25
 U 1 1 558B3941
 P 5000 5000
-F 0 "R?" V 5080 5000 40  0000 C CNN
+F 0 "R25" V 5080 5000 40  0000 C CNN
 F 1 "1k" V 5007 5001 40  0000 C CNN
 F 2 "~" V 4930 5000 30  0000 C CNN
@@
 $EndComp
 $Comp
-L R R?
+L R R26
 U 1 1 558B3947
 P 5000 5150
-F 0 "R?" V 5080 5150 40  0000 C CNN
+F 0 "R26" V 5080 5150 40  0000 C CNN
 F 1 "1k" V 5007 5151 40  0000 C CNN
 F 2 "~" V 4930 5150 30  0000 C CNN
@@
 $EndComp
 $Comp
-L VCC #PWR?
+L VCC #PWR057
 U 1 1 558B394D
 P 4100 4700
-F 0 "#PWR?" H 4100 4800 30  0001 C CNN
+F 0 "#PWR057" H 4100 4800 30  0001 C CNN
 F 1 "VCC" H 4100 4800 30  0000 C CNN
 F 2 "" H 4100 4700 60  0000 C CNN
@@
 $EndComp
 $Comp
-L R R?
+L R R27
 U 1 1 558B3964
 P 5000 5300
-F 0 "R?" V 5080 5300 40  0000 C CNN
+F 0 "R27" V 5080 5300 40  0000 C CNN
 F 1 "1k" V 5007 5301 40  0000 C CNN
 F 2 "~" V 4930 5300 30  0000 C CNN
