File: kicad/traffic_lights/traffic_lights.sch (KiCad schematic (older format))
At the start: 8 parts, among them IC1 ATMEGA328-P, IC2 74164N, IC3 74164N, IC4 74HCT595D, SW1 SW_PUSH

Commit message: added schematic
Parts:
- removed D1: LED, ~, symbol LED
- removed DS1: RC1602A-GHW-ESX, RC1602A, symbol RC1602A-GHW-ESX
- removed IC2, IC3: 74164N, 74xx-eu-DIL14, symbol 74164N
- removed IC4: 74HCT595D, 74xx-eu-SO16, symbol 74HCT595D
- added D?: LED, ~, symbol LED
- added R?: R, ~, symbol R
Connections:
- net VCC: now also D?.1 (A)
- net TC_SER_DATA: now reaches IC1.3 ((PCINT17/TXD)PD1)
- net lcd_module/LCD_LATCH_ENABLE: now reaches IC1.11 ((PCINT21/OC0B/T1)PD5)
- net lcd_module/LCD_SER_DATA: now reaches IC1.12 ((PCINT22/OC0A/AIN0)PD6)
- net SENSOR_TC_1: now reaches IC1.14 ((PCINT0/CLKO/ICP1)PB0)
- net SENSOR_TC_1: now also IC1.16 ((PCINT2/OC1B/~SS~)PB2)
- net at IC1.15 ((PCINT1/OC1A)PB1): now also R?.2
- net SENSOR_TC_3: now reaches IC1.17 ((PCINT3/OC2A/MOSI)PB3)
- net SENSOR_TC_4: now reaches IC1.18 ((PCINT4/MISO)PB4)
- net lcd_module/LCD_TRANSFER_BYTE_CLK: now reaches IC1.6 ((PCINT20/XCK/T0)PD4)
- net SR_CLK renamed TC_SER_CLK
- net TC_SER_CLK: no longer IC1.5 ((PCINT19/OC2B/INT1)PD3)
- new net: D?.2 (K), R?.1
- new net lcd_module/LCD_STORE_CLK: IC1.5 ((PCINT19/OC2B/INT1)PD3)

Commit message: update..
Parts:
- added C1, C2: C, ~, symbol C
- added X1: CRYSTAL, ~, symbol CRYSTAL
- gave numbers to parts that had none: 2
Connections:
- net labels added: XTAL1, XTAL2
- wire segments 62 -> 74
Other:
- moved on the sheet: R1, SW1
